File: Hardware/Panel.sch (EAGLE design)
At the start: 49 parts, among them J1 OUT, J2 POWER, J3 ICSP, SW1 ROTARTY_ENCODER, U1 ATTINY2313A, U2 AW9523B

Commit message: updated hardware files with latest production run
Parts:
- added C3, C4: 100n, rcl:C-EUC0402
- added H5, H6, H7, H8: 2mm, Parts:MOUNT-PAD2MM
- added J4: OUT, Class D Amp:JST-XH4
- added J5: POWER, Class D Amp:JST-XH2
- added J6: ICSP, MiniISP:MINI-ISP-LABELS
- added JP3: JUMPER-SMT_3_1-NC_TRACE_SILK, SparkFun-Jumpers:JUMPER-SMT_3_1-NC_TRACE_SILK
- added JP4: MODE, SparkFun-Jumpers:JUMPER-SMT_3_NO_SILK
- added LED17, LED18, LED19, LED20, LED21, LED22, LED23, LED24, LED25, LED26, LED27, LED28, LED29, LED30, LED31, LED32: LED-BLUE0603, BeagleBone_Blue_R3:LED-BLUE0603
- added R20, R21, R22, R23, R24, R25, R26, R27, R28, R29, R30, R31, R32, R33, R34, R35: 100, rcl:R-EU_R0402
- added R36, R37, R38: 4k7, rcl:R-EU_R0402
- added SW2: ROTARTY_ENCODER, SparkFun-Electromechanical:ROTARTY_ENCODER
- added U3: AW9523B, Parts:AW9523B
- added U4: ATTINY2313A, Parts:ATTINY2313A
Connections:
- new net N$46: J6.3, R36.1, U3.SCL, U4.PB7(UCSK/SCL/PCINT7)
- new net N$47: SW2.B, U4.PD2(CKOUT/XCK/INT0)
- new net N$48: LED28.A, R31.2
- new net N$49: LED27.A, R30.2
- new net N$50: LED26.A, R29.2
- new net N$51: LED25.A, R28.2
- new net N$52: LED24.A, R27.2
- new net N$53: LED23.A, R26.2
- new net N$54: LED22.A, R25.2
- new net N$55: LED21.A, R24.2
- new net N$56: LED32.A, R35.2
- new net N$57: LED31.A, R34.2
- new net N$58: LED30.A, R33.2
- new net N$59: LED29.A, R32.2
- new net N$60: LED20.A, R23.2
- new net N$61: LED19.A, R22.2
- new net N$62: LED18.A, R21.2
- new net N$63: LED17.A, R20.2
- new net N$64: R31.1, U3.P0_0
- new net N$65: R30.1, U3.P0_1
- new net N$66: R29.1, U3.P0_2
- new net N$67: R28.1, U3.P0_3
- new net N$68: R27.1, U3.P0_4
- new net N$69: R25.1, U3.P0_6
- new net N$70: R24.1, U3.P0_7
- new net N$71: R35.1, U3.P1_0
- new net N$72: R34.1, U3.P1_1
- new net N$73: R33.1, U3.P1_2
- new net N$74: R32.1, U3.P1_3
- new net N$75: R23.1, U3.P1_4
- new net N$76: R22.1, U3.P1_5
- new net N$77: R26.1, U3.P0_5
- new net N$78: R21.1, U3.P1_6
- new net N$79: R20.1, U3.P1_7
- new net N$80: J6.5, R38.1, U4.PA2(DW\!RESET)
- new net N$81: J6.4, R37.1, U3.SDA, U4.PB5(MOSI/DI/SDA/PCINT5)
- new net N$82: J6.1, U3.RSTN, U4.PB6(MISO/DO/PCINT6)
- new net N$83: SW2.SW-, U4.PB0(AIN0/PCINT0)
- new net N$84: J4.2, U4.PD1(TXD)
- new net N$85: J4.4, U4.PB1(AIN1/PCINT1)
- new net N$86: JP4.3, U4.PB3(OC1A/PCINT3)
- new net N$87: JP4.1, U4.PB4(OC1B/PCINT4)
- new net N$88: SW2.A, U4.PD3(INT1)
- new net N$89: J4.3, U4.PD0(RXD)
- new net N$90: JP3.2, LED17.C, LED18.C, LED19.C, LED20.C, LED21.C, LED22.C, LED23.C, LED24.C, LED25.C, LED26.C, LED27.C, LED28.C, LED29.C, LED30.C, LED31.C, LED32.C
- net +5V: now also C3.1, C4.1, J5.2, J6.2, JP3.1, R36.2, R37.2, R38.2, U3.VCC, U4.VCC
- net GND: now also C3.2, C4.2, H5.MOUNT, H6.MOUNT, H7.MOUNT, H8.MOUNT, J4.1, J5.1, J6.6, JP3.3, JP4.2, SW2.C, SW2.SW+, U3.AD0, U3.AD1, U3.GND, U3.INTN, U4.GND
